Commit message: 小圆车不带传感器

File: multi_turtlebots_sim/turtlebot3_description/urdf/mbot.xacro (robot description, xacro)
@@ -7,5 +7,5 @@
     <!-- car length0.16，camera highth0.08 -->
     <!-- <xacro:property name="camera_offset_z" value="0.10" /> -->
-    <xacro:mbot_base/>
+    <!-- <xacro:mbot_base/> -->
    <!--neck link-->
     <!-- Camera joint-->

File: multi_turtlebots_sim/turtlebot3_description/urdf/mbot_base.xacro (robot description, xacro)
@@ -7,13 +7,19 @@
     <xacro:property name="base_length" value="0.16"/>
     <!---->
+    <xacro:property name="base_mass"   value="20" />
     <xacro:property name="wheel_radius" value="0.06"/>
     <xacro:property name="wheel_length" value="0.025"/>
     <!---->
     <xacro:property name="wheel_joint_y" value="0.19"/>
-    <xacro:property name="wheel_joint_z" value="0.05"/>
+    <xacro:property name="wheel_joint_z" value="0.0"/>
     <!-- -->
-    <xacro:property name="caster_radius" value="0.015"/>
-    <!-- wheel_radius - ( base_length/2 - wheel_joint_z) -->
-    <xacro:property name="caster_joint_x" value="0.18"/>
+    <xacro:property name="caster_radius" value="0.06"/>
+    <xacro:property name="body_x" value="0.2" />
+    <xacro:property name="body_y" value="0.1" />
+    <xacro:property name="body_z" value="0.05" />
+    <xacro:property name="body_mass" value="0.5" />
+    <!--  -->
+    <xacro:property name="caster_joint_x" value="0.14"/>
+    <xacro:include filename="$(find multi_turtlebots_sim)/turtlebot3_description/urdf/mbot_base.gazebo.xacro"/>
 <!-- Defining the colors used in this robot -->
     <material name="yellow">
@@ -26,12 +32,12 @@
         <color rgba="0.75 0.75 0.75 1"/>
     </material>
-<xacro:macro name="wheel" params="prefix reflect">
-<joint name="${prefix}_wheel_joint " type="continuous"> <!--continuous360joint-->
-    <origin xyz="0 ${reflect*wheel_joint_y} ${-wheel_joint_z}" rpy="0 0 0"/>
-    <parent link="base_link"/>
-    <child link="${prefix}_wheel_link"/>
-    <axis xyz="0 1 0"/>
-</joint>
-<link name="${prefix}_wheel_link">
+    <xacro:macro name="wheel" params="prefix reflect">
+        <joint name="${prefix}_wheel_joint" type="continuous"> <!--continuous360joint-->
+            <origin xyz="0 ${reflect*wheel_joint_y} 0" rpy="0 0 0"/>
+            <parent link="base_link"/>
+            <child link="${prefix}_wheel_link"/>
+            <axis xyz="0 1 0"/>
+        </joint>
+        <link name="${prefix}_wheel_link">
             <visual>
                 <origin xyz="0 0 0" rpy="${M_PI/2} 0 0" />
@@ -41,11 +47,24 @@
                 <material name="gray" />
             </visual>
-</link>
-</xacro:macro>
+            <collision>
+                <geometry>
+                    <cylinder radius="${wheel_radius}" length = "${wheel_length}"/>
+                </geometry>
+                <origin xyz="0 0 0" rpy="${M_PI/2} 0 0" />
+            </collision>
+            <inertial>
+                <mass value="${body_mass}" />
+                <inertia ixx="${body_mass/12*(body_y*body_y+body_z*body_z)}"
+                iyy="${body_mass/12*(body_x*body_x+body_z*body_z)}"
+                izz="${body_mass/12*(body_y*body_y+body_x*body_x)}"
+                ixy="0.0" ixz="0.0" iyz="0.0"/>
+            </inertial>
+        </link>
+    </xacro:macro>
  <!-- Macro for robot caster -->
     <xacro:macro name="caster" params="prefix reflect">
         <joint name="${prefix}_caster_joint" type="continuous">
         <!---(base_length/2 + caster_radius)-->
-            <origin xyz="${reflect*caster_joint_x} 0 ${-(base_length/2 + caster_radius)}" rpy="0 0 0"/>
+            <origin xyz="${reflect*caster_joint_x} 0 0" rpy="0 0 0"/>
             <parent link="base_link"/>
             <child link="${prefix}_caster_link"/>
@@ -60,4 +79,17 @@
                 <material name="black" />
             </visual>
+            <collision>
+                <geometry>
+                    <sphere radius="${caster_radius}" />
+                </geometry>
+                <origin xyz="0 0 0"/>
+            </collision>
+            <inertial>
+                <mass value="${body_mass}" />
+                <inertia ixx="${body_mass/12*(body_y*body_y+body_z*body_z)}"
+                iyy="${body_mass/12*(body_x*body_x+body_z*body_z)}"
+                izz="${body_mass/12*(body_y*body_y+body_x*body_x)}"
+                ixy="0.0" ixz="0.0" iyz="0.0"/>
+            </inertial>
         </link>
     </xacro:macro>
@@ -65,15 +97,35 @@
         <link name="base_link">
             <visual>
-                <origin xyz="0 0 0" rpy="0 0 0" />
                 <geometry>
                     <cylinder length="${base_length}" radius="${base_radius}"/>
                 </geometry>
-                <material name="yellow" />
+                <material name="white"/>
+                <origin xyz="0 0 ${base_length/2}"/>
             </visual>
+            <collision>
+                <geometry>
+                    <cylinder length="${base_length}" radius="${base_radius}"/>
+                </geometry>
+                <origin xyz="0 0 ${base_length/2}"/>
+            </collision>
+            <inertial>
+                <mass value="${body_mass}" />
+                <inertia ixx="${body_mass/12*(body_y*body_y+body_z*body_z)}"
+                iyy="${body_mass/12*(body_x*body_x+body_z*body_z)}"
+                izz="${body_mass/12*(body_y*body_y+body_x*body_x)}"
+                ixy="0.0" ixz="0.0" iyz="0.0"/>
+            </inertial>
         </link>
+        <link name="base_footprint"/>
+        <joint name="base_joint" type="fixed">
+            <parent link="base_footprint"/>
+            <child link="base_link"/>
+            <origin xyz="0.0 0.0 0.010" rpy="0 0 0"/>
+        </joint>
         <wheel prefix="left" reflect="-1"/>
         <wheel prefix="right" reflect="1"/>
-        <caster prefix="front" reflect="-1"/>
-        <caster prefix="back" reflect="1"/>
+        <caster prefix="front" reflect="1"/>
+        <caster prefix="back" reflect="-1"/>
     </xacro:macro>
+<xacro:mbot_base/>
 </robot>
