Commit message: mbot with d415i

File: multi_turtlebots_sim/turtlebot3_description/urdf/mbot_base.gazebo.xacro (robot description, xacro)
@@ -32,3 +32,65 @@
         </plugin>
     </gazebo>
+    <gazebo reference="camera_link_fake">
+      	    <sensor type="depth" name="camera_D415">
+                <updateRate>30.0</updateRate>
+                <camera name="head">
+                    <image>
+                    <width>1280</width>
+                    <height>720</height>
+                    <format>R8G8B8</format>
+                    </image>
+                    <clip>
+                    <near>0.3</near>
+                    <far>10</far>
+                    </clip>
+                    <noise>
+                    <type>gaussian</type>
+                    <!-- Noise is sampled independently per pixel on each frame.
+                        That pixel's noise value is added to each of its color
+                        channels, which at that point lie in the range [0,1]. -->
+                    <mean>0.0</mean>
+                    <stddev>0.005</stddev>
+                    </noise>
+                </camera>
+                <plugin name="camera_D415_camera_controller" filename="libgazebo_ros_openni_kinect.so">
+                    <alwaysOn>true</alwaysOn>
+                    <updateRate>0.0</updateRate>
+                    <cameraName>camera</cameraName>
+                    <imageTopicName>rgb/image_raw</imageTopicName>
+                    <depthImageTopicName>depth/image_raw</depthImageTopicName>
+                    <pointCloudTopicName>depth/points</pointCloudTopicName>
+                    <cameraInfoTopicName>rgb/camera_info</cameraInfoTopicName>
+                    <depthImageCameraInfoTopicName>depth/camera_info</depthImageCameraInfoTopicName>
+                    <frameName>camera_link_optical</frameName>
+                    <baseline>0.1</baseline>
+                    <distortion_k1>0.0</distortion_k1>
+                    <distortion_k2>0.0</distortion_k2>
+                    <distortion_k3>0.0</distortion_k3>
+                    <distortion_t1>0.0</distortion_t1>
+                    <distortion_t2>0.0</distortion_t2>
+                    <pointCloudCutoff>0.05</pointCloudCutoff>
+                    <rangeMax>4.0</rangeMax>
+                </plugin>
+         </sensor>
+    </gazebo>
+    <gazebo reference="imu_link">
+        <gravity>true</gravity>
+        <sensor name="imu_sensor" type="imu">
+        <always_on>true</always_on>
+        <update_rate>100</update_rate>
+        <visualize>true</visualize>
+        <topic>__default_topic__</topic>
+        <plugin filename="libgazebo_ros_imu_sensor.so" name="imu_plugin">
+            <topicName>imu</topicName>
+            <bodyName>imu_link</bodyName>
+            <updateRateHZ>10.0</updateRateHZ>
+            <gaussianNoise>0.0</gaussianNoise>
+            <xyzOffset>0 0 0</xyzOffset>
+            <rpyOffset>0 0 0</rpyOffset>
+            <frameName>imu_link</frameName>
+        </plugin>
+        <pose>0 0 0 0 0 0</pose>
+        </sensor>
+    </gazebo>
 </robot>

File: multi_turtlebots_sim/turtlebot3_description/urdf/mbot_base.xacro (robot description, xacro)
@@ -22,4 +22,6 @@
     <xacro:property name="caster_joint_x" value="0.14"/>
     <xacro:include filename="$(find multi_turtlebots_sim)/turtlebot3_description/urdf/mbot_base.gazebo.xacro"/>
+    <xacro:include filename="$(find multi_turtlebots_sim)/turtlebot3_description/urdf/mbot_camera.xacro"/>
+    <xacro:realsense/>
 <!-- Defining the colors used in this robot -->
     <material name="yellow">

File: multi_turtlebots_sim/turtlebot3_description/urdf/mbot_camera.xacro (robot description, xacro)
@@ -2,6 +2,6 @@
 <robot xmlns:xacro="http://www.ros.org/wiki/xacro" name="camera">
     <!--prefix:=camera camera-->
-    <xacro:macro name="usb_camera" params="prefix:=camera">
-        <link name="${prefix}_link">
+    <xacro:macro name="realsense">
+        <!-- <link name="${prefix}_link">
             <visual>
                 <origin xyz=" 0 0 0 " rpy="0 0 0" />
@@ -11,5 +11,57 @@
                 <material name="black"/>
             </visual>
+        </link> -->
+          <!-- Camera -->
+        <link name="camera_link">
+            <collision>
+            <origin xyz="0 0 0" rpy="0 0 0"/>
+            <geometry>
+                <box size="0.1 0.1 0.1"/>
+            </geometry>
+            </collision>
+            <visual>
+            <origin xyz="0 0 0" rpy="0 0 1.5708"/>
+            <geometry>
+                <!--<mesh filename="package://robot_sim_demo/models/meshes/xtion_pro_camera.dae" />-->
+                <mesh filename="package://multi_turtlebots_sim/turtlebot3_description/meshes/sensors/realsense.obj" />
+            </geometry>
+            </visual>
+            <inertial>
+            <mass value="1e-5" />
+            <origin xyz="0 0 0" rpy="0 0 0"/>
+            <inertia ixx="1e-6" ixy="0" ixz="0" iyy="1e-6" iyz="0" izz="1e-6" />
+            </inertial>
         </link>
+        <joint name="camera_joint" type="fixed">
+            <axis xyz="0 0.5 0" />
+            <origin xyz="0 0 0.20" rpy="0 0 -1.5708"/>
+            <parent link="base_link"/>
+            <child link="camera_link"/>
+        </joint>
+        <!-- generate an optical frame http://www.ros.org/reps/rep-0103.html#suffix-frames
+            so that ros and opencv can operate on the camera frame correctly -->
+             <!-- these values have to be these values otherwise the gazebo camera image
+                won't be aligned properly with the frame it is supposedly originating from -->
+        <joint name="camera_fake_joint" type="fixed">
+            <origin xyz="0 0 0" rpy="0 0 1.5708"/>
+            <parent link="camera_link"/>
+            <child link="camera_link_fake"/>
+        </joint>
+        <link name="camera_link_fake">
+        </link>
+        <joint name="camera_optical_joint" type="fixed">
+            <origin xyz="0 0 0" rpy="-1.5708 0 -1.5708"/>
+            <parent link="camera_link_fake"/>
+            <child link="camera_link_optical"/>
+        </joint>
+        <link name="camera_link_optical">
+        </link>
+        <link name="imu_link"/>
+        <joint name="base_to_imu" type="fixed">
+            <axis rpy="0 0 0" xyz="0 0 0"/>
+            <parent link="camera_link"/>
+            <child link="imu_link"/>
+            <origin rpy="0 0 0" xyz="0 0 .2"/>
+        </joint>
     </xacro:macro>
 </robot>

Commit message: 添加带liar

File: multi_turtlebots_sim/turtlebot3_description/urdf/mbot_base.gazebo.xacro (robot description, xacro)
@@ -42,6 +42,6 @@
                     </image>
                     <clip>
-                    <near>0.3</near>
-                    <far>10</far>
+                    <near>0.01</near>
+                    <far>300</far>
                     </clip>
                     <noise>
@@ -64,5 +64,5 @@
                     <depthImageCameraInfoTopicName>depth/camera_info</depthImageCameraInfoTopicName>
                     <frameName>camera_link_optical</frameName>
-                    <baseline>0.1</baseline>
+                    <baseline>0.01</baseline>
                     <distortion_k1>0.0</distortion_k1>
                     <distortion_k2>0.0</distortion_k2>
@@ -70,6 +70,8 @@
                     <distortion_t1>0.0</distortion_t1>
                     <distortion_t2>0.0</distortion_t2>
-                    <pointCloudCutoff>0.05</pointCloudCutoff>
-                    <rangeMax>4.0</rangeMax>
+                    <pointCloudCutoff>0.0005</pointCloudCutoff>
+                    <pointCloudCutoffMax>30.0</pointCloudCutoffMax>
+                    <rangeMin>0.00005</rangeMin>
+                    <rangeMax>40.0</rangeMax>
                 </plugin>
          </sensor>
@@ -94,3 +96,34 @@
         </sensor>
     </gazebo>
+    <gazebo reference="lidar_link">
+    <sensor type="ray" name="laser">
+      <pose>0 0 0 0 0 0</pose>
+      <visualize>false</visualize>
+      <update_rate>20</update_rate>
+      <ray>
+        <scan>
+          <horizontal>
+            <samples>810</samples>
+            <resolution>1</resolution>
+            <min_angle>-3.1415926</min_angle>
+            <max_angle>3.1415926</max_angle>
+          </horizontal>
+        </scan>
+        <range>
+          <min>0.10</min>
+          <max>20.0</max>
+          <resolution>0.01</resolution>
+        </range>
+        <noise>
+          <type>gaussian</type>
+          <mean>0.0</mean>
+          <stddev>0.01</stddev>
+        </noise>
+      </ray>
+      <plugin name="gazebo_ros_head_hokuyo_controller" filename="libgazebo_ros_laser.so">
+        <topicName>scan</topicName>
+        <frameName>lidar_link</frameName>
+      </plugin>
+    </sensor>
+    </gazebo>
 </robot>

File: multi_turtlebots_sim/turtlebot3_description/urdf/mbot_base.xacro (robot description, xacro)
@@ -21,7 +21,4 @@
     <!--  -->
     <xacro:property name="caster_joint_x" value="0.14"/>
-    <xacro:include filename="$(find multi_turtlebots_sim)/turtlebot3_description/urdf/mbot_base.gazebo.xacro"/>
-    <xacro:include filename="$(find multi_turtlebots_sim)/turtlebot3_description/urdf/mbot_camera.xacro"/>
-    <xacro:realsense/>
 <!-- Defining the colors used in this robot -->
     <material name="yellow">
@@ -125,9 +122,8 @@
             <origin xyz="0.0 0.0 0.010" rpy="0 0 0"/>
         </joint>
-        <wheel prefix="left" reflect="-1"/>
-        <wheel prefix="right" reflect="1"/>
+        <wheel prefix="left" reflect="1"/>
+        <wheel prefix="right" reflect="-1"/>
         <caster prefix="front" reflect="1"/>
         <caster prefix="back" reflect="-1"/>
     </xacro:macro>
-<xacro:mbot_base/>
 </robot>

File: multi_turtlebots_sim/turtlebot3_description/urdf/mbot_ob.xacro (robot description, xacro)
@@ -1,4 +1,4 @@
 <?xml version="1.0"?>
-<robot name="arm" xmlns:xacro="http://www.ros.org/wiki/xacro">
+<robot name="ob" xmlns:xacro="http://www.ros.org/wiki/xacro">
     <xacro:include filename="$(find multi_turtlebots_sim)/turtlebot3_description/urdf/mbot_base.xacro" />
     <xacro:include filename="$(find multi_turtlebots_sim)/turtlebot3_description/urdf/mbot_base.gazebo.xacro"/>
@@ -6,3 +6,4 @@
     <xacro:realsense/>
     <xacro:mbot_base/>
+    <xacro:rplidarA2 name="lidar_link" ros_topic="scan" />
 </robot>

File: multi_turtlebots_sim/turtlebot3_description/urdf/mbot_property.xacro (robot description, xacro)
@@ -1,4 +1,4 @@
 <?xml version="1.0"?>
-<robot xmlns:xacro="http://www.ros.org/wiki/xacro" name="camera">
+<robot xmlns:xacro="http://www.ros.org/wiki/xacro" name="property">
     <!--prefix:=camera camera-->
     <xacro:macro name="realsense">
@@ -35,5 +35,5 @@
         <joint name="camera_joint" type="fixed">
             <axis xyz="0 0.5 0" />
-            <origin xyz="0 0 0.20" rpy="0 0 -1.5708"/>
+            <origin xyz="0 0 0.250" rpy="0 0 -1.5708"/>
             <parent link="base_link"/>
             <child link="camera_link"/>
@@ -65,3 +65,40 @@
         </joint>
     </xacro:macro>
+    <xacro:macro name="rplidarA2" params="name ros_topic">
+    <xacro:sick_tim name="${name}" ros_topic="${ros_topic}"
+      length="0.06" width="0.06" height="0.079" mass="0.150" z_offset="0.33"
+      min_range="0.2" max_range="8.0"
+      mesh="package://multi_turtlebots_sim/turtlebot3_description/meshes/sensors/rplidar.dae" />
+    </xacro:macro>
+    <xacro:macro name="sick_tim" params="name ros_topic length width height mass z_offset min_range max_range mesh">
+    <!-- z_offset: distance between base plate and laser center (= center of mesh) -->
+    <joint name="${name}_joint" type="fixed">
+      <parent link="base_link" />
+      <child link="${name}" />
+      <origin rpy="0 0 0" xyz="0 0 ${z_offset}"/>
+    </joint>
+    <link name="${name}">
+      <visual>
+        <geometry>
+          <mesh filename="${mesh}" />
+        </geometry>
+        <material name="lightblue">
+          <color rgba=".5 .5 .7 .8" />
+        </material>
+      </visual>
+      <collision>
+        <geometry>
+          <mesh filename="${mesh}" />
+        </geometry>
+      </collision>
+      <inertial>
+        <mass value="${mass}" />
+        <origin xyz="0 0 -0.026" />
+        <inertia ixx="${0.0833333 * mass * (width * width + height * height)}" ixy="0.0" ixz="0.0"
+          iyy="${0.0833333 * mass * (length * length + height * height)}" iyz="0.0"
+          izz="${0.0833333 * mass * (length * length + width * width)}" />
+      </inertial>
+    </link>
+    <!--update_rate=15.0-->
+    </xacro:macro>
 </robot>
